File: tranz330_cpuboard_periph.sch (KiCad schematic (older format))
At the start: 22 parts, among them P1 CONN_01X20, P4 CONN_01X08, P5 CONN_01X06, U11 74HC04, U15 Z80DART, U2 M6242B, U20 DS1489, U28 DS14C88, U30 73K212AL, U4 Z80CTC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

Commit message: Add interrupt enable chain, note on reset, PDF version
Parts:
- gave numbers to parts that had none: 1
Connections:
- net +5V: now also U9.24 (IEI)
- net /INT: now also U4.12 (/INT)
- net CTC_IEO: now reaches U15.6 (IEI)
- net CTC_IEO: now also U4.11 (IEO)
- net VEE: now reaches U28.1 (V-)
- net VEE: now also P1.18 (P18)
- net PIO_IEO: now reaches U9.22 (IEO)
- net PIO_IEO: now also U4.13 (IEI)
Changed lines of the file:
@@
 	9850 6150 9850 6200
-$Comp
-L GND #PWR?
-U 1 1 596228F5
-P 7600 3750
-F 0 "#PWR?" H 7600 3500 50  0001 C CNN
-F 1 "GND" H 7600 3600 50  0000 C CNN
-F 2 "" H 7600 3750 50  0000 C CNN
-F 3 "" H 7600 3750 50  0000 C CNN
-	1    7600 3750
-	1    0    0    -1
-$EndComp
 $Comp
 L +5V #PWR?
@@
 NoConn ~ 8250 2000
 NoConn ~ 8250 2100
-NoConn ~ 7600 3800
-$Comp
-L 74HC04 U?
+$Comp
+L 74HC04 U11
 U 2 1 5962CF20
 P 950 3000
-F 0 "U?" H 1100 3100 50  0000 C CNN
+F 0 "U11" H 1100 3100 50  0000 C CNN
 F 1 "74HC04" H 1150 2900 50  0000 C CNN
 F 2 "" H 950 3000 50  0000 C CNN
@@
 Wire Wire Line
 	850  4800 1050 4800
+Text GLabel 9100 5700 0    39   Output ~ 0
+CTC_IEO
+Wire Wire Line
+	9200 5700 9100 5700
+Text GLabel 850  5400 0    39   Input ~ 0
+CTC_IEO
+Wire Wire Line
+	850  5400 1050 5400
+Text GLabel 6750 3300 0    39   Output ~ 0
+PIO_IEO
+Wire Wire Line
+	6750 3300 6950 3300
+$Comp
+L +5V #PWR?
+U 1 1 596C806F
+P 6400 3100
+F 0 "#PWR?" H 6400 2950 50  0001 C CNN
+F 1 "+5V" H 6400 3240 50  0000 C CNN
+F 2 "" H 6400 3100 50  0000 C CNN
+F 3 "" H 6400 3100 50  0000 C CNN
+	1    6400 3100
+	1    0    0    -1
+$EndComp
+Wire Wire Line
+	6400 3100 6400 3200
+Wire Wire Line
+	6400 3200 6950 3200
+Text GLabel 9100 5600 0    39   Input ~ 0
+PIO_IEO
+Wire Wire Line
+	9100 5600 9200 5600
+NoConn ~ 1050 5500
+Text GLabel 9100 5800 0    39   Input ~ 0
+/INT
+Wire Wire Line
+	9100 5800 9200 5800
+$Comp
+L VEE #PWR?
+U 1 1 596CA02C
+P 3050 7600
+F 0 "#PWR?" H 3050 7450 50  0001 C CNN
+F 1 "VEE" H 3050 7750 50  0000 C CNN
+F 2 "" H 3050 7600 50  0000 C CNN
+F 3 "" H 3050 7600 50  0000 C CNN
+	1    3050 7600
+	-1   0    0    1
+$EndComp
+Wire Wire Line
+	3050 7550 3050 7600
+$Comp
+L VEE #PWR?
+U 1 1 596CA40F
+P 9200 2800
+F 0 "#PWR?" H 9200 2650 50  0001 C CNN
+F 1 "VEE" H 9200 2950 50  0000 C CNN
+F 2 "" H 9200 2800 50  0000 C CNN
+F 3 "" H 9200 2800 50  0000 C CNN
+	1    9200 2800
+	-1   0    0    1
+$EndComp
+Wire Wire Line
+	9200 2800 9200 2750
+Wire Wire Line
+	9200 2750 9850 2750
+$Comp
+L GND #PWR?
+U 1 1 596228F5
+P 7600 3750
+F 0 "#PWR?" H 7600 3500 50  0001 C CNN
+F 1 "GND" H 7600 3600 50  0000 C CNN
+F 2 "" H 7600 3750 50  0000 C CNN
+F 3 "" H 7600 3750 50  0000 C CNN
+	1    7600 3750
+	1    0    0    -1
+$EndComp
 $EndSCHEMATC

Commit message: Fix the modem xtal frequency
Parts:
- Y4: value 16.96K -> 11.0592M
Changed lines of the file:
@@
 U 1 1 59616EC8
 P 2850 2300
-F 0 "Y4" H 2850 2450 50  0000 C CNN
-F 1 "16.96K" H 2850 2150 50  0000 C CNN
+F 0 "Y4" H 2850 2150 50  0000 C CNN
+F 1 "11.0592M" H 2900 2450 50  0000 C CNN
 F 2 "" H 2850 2300 50  0000 C CNN
 F 3 "" H 2850 2300 50  0000 C CNN
@@
 U 1 1 596174B3
 P 2850 2650
-F 0 "C57" H 2875 2750 50  0000 L CNN
+F 0 "C57" H 2700 2750 50  0000 L CNN
 F 1 "C" H 2875 2550 50  0000 L CNN
 F 2 "" H 2888 2500 50  0000 C CNN
