File: tranz330_re.sch (KiCad schematic (older format))
At the start: 23 parts, among them Q1 2N7008, U11 74HC04, U14 74LS10, U16 74HC74, U5 62256, U6 27C256, U7 Z80A, U8 74LS138, Y3 7.15909

Commit message: Add interrupt enable chain, note on reset, PDF version
Parts:
- U14: value 74LS10 -> 74HC10
Other:
- note added: "/RESET is generated\nfrom the L387A regulator's \nreset output (U27 pin 2)\n"
Changed lines of the file:
@@
 P 2600 5200
 F 0 "U14" H 2600 5250 50  0000 C CNN
-F 1 "74LS10" H 2600 5150 50  0000 C CNN
+F 1 "74HC10" H 2600 5150 50  0000 C CNN
 F 2 "" H 2600 5200 50  0000 C CNN
 F 3 "" H 2600 5200 50  0000 C CNN
@@
 P 2600 5800
 F 0 "U14" H 2600 5850 50  0000 C CNN
-F 1 "74LS10" H 2600 5750 50  0000 C CNN
+F 1 "74HC10" H 2600 5750 50  0000 C CNN
 F 2 "" H 2600 5800 50  0000 C CNN
 F 3 "" H 2600 5800 50  0000 C CNN
@@
 P 7100 5600
 F 0 "U14" H 7100 5650 50  0000 C CNN
-F 1 "74LS10" H 7100 5550 50  0000 C CNN
+F 1 "74HC10" H 7100 5550 50  0000 C CNN
 F 2 "" H 7100 5600 50  0000 C CNN
 F 3 "" H 7100 5600 50  0000 C CNN
@@
 Text Notes 9400 1800 0    60   ~ 0
 DART\nPIO\nCTC\nSerial\nModem\nRTC
+Text Notes 6300 2900 0    39   ~ 0
+/RESET is generated\nfrom the L387A regulator's \nreset output (U27 pin 2)\n
 $EndSCHEMATC

Commit message: Fix /RTSB, better PDF output, trace missing DART and modem pins
Other:
- note added: "/RESET is generated from the\nL387A regulator's reset output\n(U27 pin 2) if +5V is not stable.\nQ1 prevents the RAM from being\nwritten with garbage when +5V\nis coming up or going down."
- note added: "VMEM is supplied from a diode-OR\nof the 3V lithium cell at B1 and +5V.\nRAM contents are always retained\nwhen power is off, so watch those\nuninitialized variables.\n"
- note removed: "/RESET is generated\nfrom the L387A regulator's \nreset output (U27 pin 2)\n"
Changed lines of the file:
@@
 encoding utf-8
 Sheet 1 2
-Title ""
-Date ""
-Rev ""
+Title "Top Level - CPU, RAM, clock, I/O decode"
+Date "2017-07-24"
+Rev "0.5"
 Comp ""
-Comment1 ""
+Comment1 "VeriFone Tranz 330 reverse engineered schematic"
 Comment2 ""
 Comment3 ""
@@
 Entry Wire Line
 	7700 5200 7800 5300
-Text GLabel 7600 4800 0    59   BiDi ~ 0
+Text GLabel 7600 4800 0    59   Input ~ 0
 A
 Text Label 7800 5100 0    39   ~ 0
@@
 DART\nPIO\nCTC\nSerial\nModem\nRTC
 Text Notes 6300 2900 0    39   ~ 0
-/RESET is generated\nfrom the L387A regulator's \nreset output (U27 pin 2)\n
+/RESET is generated from the\nL387A regulator's reset output\n(U27 pin 2) if +5V is not stable.\nQ1 prevents the RAM from being\nwritten with garbage when +5V\nis coming up or going down.
+Text Notes 5500 2100 0    39   ~ 0
+VMEM is supplied from a diode-OR\nof the 3V lithium cell at B1 and +5V.\nRAM contents are always retained\nwhen power is off, so watch those\nuninitialized variables.\n
 $EndSCHEMATC
